File: PCB/plant-monitor-pot.kicad_pcb (KiCad board)
At the start: 2 copper layers, 60.7 x 45.8 mm, 75 parts, among them J1 TYPE-C-31-M-12, J10 DATA, J11 GND, J12 VCC_3V3, J13 DATA, J14 GND, J2 VCC_4V, J3 GND, J6 DATA, J7 VCC_3V3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

Commit message: new pcb
Parts:
- removed D8: SB220, Diode_SMD:D_0402_1005Metric
- added D10: SS24, Diode_SMD:D_SMA, F.Cu at (105.5, 73.0)
- S1: value EG1270 -> EG1247; footprint EG1270:SW_EG1270 -> EG1247:SW_EG1247
- moved e 7.02 mm to (112.0, 73.0)
- moved R17 0.50 mm to (121.0, 70.0)
- moved S1 0.40 mm to (139.8, 75.5)
Routing:
- net 5V+: track 54.8 -> 58.1 mm
- net OUT+: track 68.2 -> 70.7 mm
- net ESP_3V3: track 137.1 -> 135.7 mm
- net A1: track 67.9 -> 68.6 mm
Other:
- board text added: "+ -"
- board text added: "+ - SOLAR"
- board text added: "BOOT"
- board text added: "RST"
- board text removed: "BAT+ -"
- board text removed: "SOLAR + -"
